File: input_output_filter.kicad_sch (KiCad schematic)
At the start: 46 parts, among them J1 XLR3_AudioJack3_Combo_Ground, J2 NC3MAH, J3 NC3MAH, J4 NC3MAH, J5 NC3MAH, J6 XLR3_AudioJack3_Combo_Ground, SW2 SW_SPST, SW3 SW_SPST, SW4 SW_SPST, SW5 SW_SPST, SW6 SW_SPST, SW7 SW_SPST, T1 Transformer_Audio, T2 Transformer_Audio, T3 Transformer_Audio, T4 Transformer_Audio

Commit message: aggiunto filtro PLL_LF Adau
Parts:
- renumbered J2 to J1, J3 to J2, J4 to J3, J5 to J4, J6 to J5, J1 to J6
Connections:
- net ADC0: now also R12.1; no longer R10.1
- net ADC1: now also R10.1; no longer R12.1
Changed lines of the file:
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@@
 		)
 	)
-	(label "ADC1"
+	(label "ADC0"
 		(at 274.32 39.37 0)
 		(effects
@@
 		)
 	)
-	(label "ADC0"
+	(label "ADC1"
 		(at 274.32 114.3 0)
 		(effects
@@
 		(dnp no)
 		(fields_autoplaced yes)
-		(property "Reference" "J1"
+		(property "Reference" "J6"
 			(at 198.12 100.3299 90)
 			(show_name no)
@@
 			(project "DSP-hw"
 				(path "/665533d7-60b6-4e6a-837a-6e08e6e15a4b"
-					(reference "J1")
+					(reference "J6")
 					(unit 1)
 				)
@@
 		(dnp no)
 		(fields_autoplaced yes)
-		(property "Reference" "J4"
+		(property "Reference" "J3"
 			(at 146.05 96.5199 90)
 			(show_name no)
@@
 			(project "DSP-hw"
 				(path "/665533d7-60b6-4e6a-837a-6e08e6e15a4b"
-					(reference "J4")
+					(reference "J3")
 					(unit 1)
 				)
@@
 		(dnp no)
 		(fields_autoplaced yes)
-		(property "Reference" "J2"
+		(property "Reference" "J1"
 			(at 144.78 29.2099 90)
 			(show_name no)
@@
 			(project "DSP-hw"
 				(path "/665533d7-60b6-4e6a-837a-6e08e6e15a4b"
-					(reference "J2")
+					(reference "J1")
 					(unit 1)
 				)
@@
 		(dnp no)
 		(fields_autoplaced yes)
-		(property "Reference" "J6"
+		(property "Reference" "J5"
 			(at 198.12 25.3999 90)
 			(show_name no)
@@
 			(project "DSP-hw"
 				(path "/665533d7-60b6-4e6a-837a-6e08e6e15a4b"
-					(reference "J6")
+					(reference "J5")
 					(unit 1)
 				)
@@
 		(dnp no)
 		(fields_autoplaced yes)
-		(property "Reference" "J1"
+		(property "Reference" "J6"
 			(at 203.835 119.38 0)
 			(show_name no)
@@
 			(project "DSP-hw"
 				(path "/665533d7-60b6-4e6a-837a-6e08e6e15a4b"
-					(reference "J1")
+					(reference "J6")
 					(unit 2)
 				)
@@
 		(dnp no)
 		(fields_autoplaced yes)
-		(property "Reference" "J3"
+		(property "Reference" "J2"
 			(at 146.05 62.2299 90)
 			(show_name no)
@@
 			(project "DSP-hw"
 				(path "/665533d7-60b6-4e6a-837a-6e08e6e15a4b"
-					(reference "J3")
+					(reference "J2")
 					(unit 1)
 				)
@@
 		(dnp no)
 		(fields_autoplaced yes)
-		(property "Reference" "J5"
+		(property "Reference" "J4"
 			(at 146.05 134.6199 90)
 			(show_name no)
@@
 			(project "DSP-hw"
 				(path "/665533d7-60b6-4e6a-837a-6e08e6e15a4b"
-					(reference "J5")
+					(reference "J4")
 					(unit 1)
 				)
@@
 		(dnp no)
 		(fields_autoplaced yes)
-		(property "Reference" "J6"
+		(property "Reference" "J5"
 			(at 203.835 44.45 0)
 			(show_name no)
@@
 			(project "DSP-hw"
 				(path "/665533d7-60b6-4e6a-837a-6e08e6e15a4b"
-					(reference "J6")
+					(reference "J5")
 					(unit 2)
 				)

Commit message: sostituito micro esp32 a stm32
Parts:
- removed SW2, SW3, SW4, SW5: SW_SPST, Button_Switch_THT:SW_DIP_SPSTx01_Slide_9.78x4.72mm_W7.62mm_P2.54mm, symbol Switch:SW_SPST
- removed T1, T2, T3, T4: Transformer_Audio, symbol Device:Transformer_Audio
Connections:
- net GND: now also J1.1, J1.3, J1.G, J2.1, J2.3, J2.G, J3.1, J3.3, J3.G, J4.1, J4.3, J4.G
- net at J3.2: now also C33.1, C34.1, R19.1, R20.1, R21.1
- net at J1.2: now also C27.1, C28.1, R13.1, R14.1, R15.1
- net at C36.1, C37.1, R22.1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: now also J4.2
- net at C30.1, C31.1, R16.1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: now also J2.2
Other:
- moved on the sheet: J1, J2, J3, J4
