File: input_output_filter.kicad_sch (KiCad schematic)
At the start: 39 parts, among them J1 NC3MAH, J2 NC3MAH, J3 NC3MAH, J4 NC3MAH, J5 XLR3_AudioJack3_Combo_Ground, J6 XLR3_AudioJack3_Combo_Ground, SW6 SW_SPST, SW7 SW_SPST, U5 IH0515S

Commit message: errore alla coca
Parts:
- removed C27, C30, C33, C36: 56n, Capacitor_SMD:C_0603_1608Metric, symbol Device:C
- removed R14, R17, R20, R23: 47k, Resistor_SMD:R_0603_1608Metric, symbol Device:R
- removed U5: IH0515S, Converter_DCDC:Converter_DCDC_XP_POWER-IHxxxxS_THT, symbol Converter_DCDC:IH0515S
- added J10, J11: AudioJack3, Connector_Audio:Jack_3.5mm_CUI_SJ1-3523N_Horizontal, symbol Connector_Audio:AudioJack3
- C28, C31, C34, C37: value 56n -> 100n
- R15, R18, R21, R24: value 47k -> 22k
Connections:
- net GND: now also J10.S, J11.S
- net at C37.1, J4.2, R22.1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: now also J11.R
- net at C34.1, J3.2, R19.1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: now also J11.T
- net at C31.1, J2.2, R16.1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: now also J10.R
- net at C28.1, J1.2, R13.1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: now also J10.T
Other:
- moved on the sheet: C28, C31, C34, C37, R15, R18, R21, R24

Commit message: recuperata versione di ieri
Parts:
- C24, C25, C26, C29, C32: footprint Capacitor_SMD:C_0603_1608Metric -> Capacitor_SMD:C_1210_3225Metric
Changed lines of the file:
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@@
 			)
 		)
-		(property "Footprint" "Capacitor_SMD:C_0603_1608Metric"
+		(property "Footprint" "Capacitor_SMD:C_1210_3225Metric"
 			(at 33.02 26.9748 0)
 			(hide yes)
@@
 			)
 		)
-		(property "Footprint" "Capacitor_SMD:C_0603_1608Metric"
+		(property "Footprint" "Capacitor_SMD:C_1210_3225Metric"
 			(at 254 113.3348 0)
 			(hide yes)
@@
 			)
 		)
-		(property "Footprint" "Capacitor_SMD:C_0603_1608Metric"
+		(property "Footprint" "Capacitor_SMD:C_1210_3225Metric"
 			(at 34.29 94.2848 0)
 			(hide yes)
@@
 			)
 		)
-		(property "Footprint" "Capacitor_SMD:C_0603_1608Metric"
+		(property "Footprint" "Capacitor_SMD:C_1210_3225Metric"
 			(at 254 38.4048 0)
 			(hide yes)
@@
 			)
 		)
-		(property "Footprint" "Capacitor_SMD:C_0603_1608Metric"
+		(property "Footprint" "Capacitor_SMD:C_1210_3225Metric"
 			(at 34.29 59.9948 0)
 			(hide yes)

Commit message: routing iniziale
Parts:
- C35: footprint Capacitor_SMD:C_0603_1608Metric -> Capacitor_SMD:C_1210_3225Metric
Changed lines of the file:
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@@
 			)
 		)
-		(property "Footprint" "Capacitor_SMD:C_0603_1608Metric"
+		(property "Footprint" "Capacitor_SMD:C_1210_3225Metric"
 			(at 34.29 132.3848 0)
 			(hide yes)

Commit message: cambiato connettori jack
Parts:
- J10, J11: footprint Connector_Audio:Jack_3.5mm_CUI_SJ1-3523N_Horizontal -> Connector_Audio:Jack_3.5mm_Lumberg_1503_07_Horizontal
Changed lines of the file:
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@@
 			)
 		)
-		(property "Footprint" "Connector_Audio:Jack_3.5mm_CUI_SJ1-3523N_Horizontal"
+		(property "Footprint" "Connector_Audio:Jack_3.5mm_Lumberg_1503_07_Horizontal"
 			(at 129.54 50.8 0)
 			(hide yes)
@@
 			)
 		)
-		(property "Footprint" "Connector_Audio:Jack_3.5mm_CUI_SJ1-3523N_Horizontal"
+		(property "Footprint" "Connector_Audio:Jack_3.5mm_Lumberg_1503_07_Horizontal"
 			(at 130.81 120.65 0)
 			(hide yes)

Commit message: modifiche suggerite da osti
Parts:
- added H1, H2, H3, H4: MountingHole, MountingHole:MountingHole_3.2mm_M3_Pad_Via, symbol Mechanical:MountingHole

Commit message: bom completata
Parts:
- C24, C25, C26, C29, C32, C35: footprint Capacitor_SMD:C_1210_3225Metric -> Capacitor_SMD:C_0805_2012Metric
- J10, J11: footprint Connector_Audio:Jack_3.5mm_Lumberg_1503_07_Horizontal -> Connector_Audio:Jack_3.5mm_CUI_SJ1-3523N_Horizontal

Commit message: pulito lo schematico e fatto dei check
Parts:
- added H5, H6, H7, H8: MountingHole, MountingHole:MountingHole_2.2mm_M2_Pad_Via, symbol Mechanical:MountingHole
- added J12: Conn_01x06_Socket, Connector_PinHeader_2.54mm:PinHeader_1x06_P2.54mm_Vertical, symbol Connector:Conn_01x06_Socket
Connections:
- net GND: now also J12.6 (Pin_6)
- net 1 Hot: now reaches C24.1, J6.2, J6.T, R9.1
- net 1 Hot: now also J12.3 (Pin_3)
- net 1 Cold: now reaches J6.3, J6.R, SW6.2 (B)
- net 1 Cold: now also J12.2 (Pin_2)
- net 0 Hot: now reaches C25.1, J5.2, J5.T, R11.1
- net 0 Hot: now also J12.5 (Pin_5)
- net 0 Cold: now reaches J5.3, J5.R, SW7.2 (B)
- net 0 Cold: now also J12.4 (Pin_4)
- new net +5V: J12.1 (Pin_1)
Other:
- note added: "Analog input"
- note added: "Analog output"
- note added: "Phantom 48v output"
- note added: "Phantom mounting hole"
- moved on the sheet: C26, C28, C29, C31, C32, C34, C35, C37, H1, H2, H3, H4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
