File: DSP-hw.kicad_sch (KiCad schematic)
At the start: 50 parts, among them Q1 BC327, Q2 AO3400A, SW1 SW_Push, SW8 SW_Push, U1 ADAU1701, U2 CAT24C256, U3 AMS1117-3.3, Y1 12.228M

Commit message: recuperata versione di ieri
Parts:
- removed C1, C6: 100n, Capacitor_SMD:C_0603_1608Metric, symbol Device:C
- removed C2, C5: 10u, Capacitor_SMD:C_0603_1608Metric, symbol Device:C
- C10, C11, C13, C15, C17, C4, C8: footprint Capacitor_SMD:C_0603_1608Metric -> Capacitor_SMD:C_0805_2012Metric
- C19, C20: footprint Capacitor_SMD:C_0603_1608Metric -> Capacitor_THT:C_Radial_D5.0mm_H11.0mm_P2.00mm
Connections:
- net +3V3: no longer Q1.2 (B), R1.1, U1.17 (VDRIVE)
- new net: Q1.2 (B), R1.1, U1.17 (VDRIVE)
