File: DSP-hw.kicad_sch (KiCad schematic)
At the start: 46 parts, among them Q1 BC327, Q2 AO3400A, SW1 SW_Push, SW8 SW_Push, U1 ADAU1701, U2 CAT24C256, U3 AMS1117-3.3, Y1 12.228M

Commit message: aggiunto oscillatore allo schematico
Parts:
- added C27: 100n, Capacitor_SMD:C_0603_1608Metric, symbol Device:C
- C17: value 10u -> 47u; footprint Capacitor_SMD:C_0805_2012Metric -> Capacitor_THT:C_Radial_D5.0mm_H11.0mm_P2.00mm
- C7: value 1u -> 100n
Connections:
- net GND: now also C27.1
- net at C7.2, C8.2, U1.34 (PVDD)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: now also C27.2
- no-connect marks 0 -> 3
Changed lines of the file:
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@@
 	)
 	(junction
+		(at 212.09 63.5)
+		(diameter 0)
+		(color 0 0 0 0)
+	)
+	(junction
 		(at 210.82 138.43)
 		(diameter 0)
@@
 		(color 0 0 0 0)
 	)
+	(junction
+		(at 191.77 63.5)
+		(diameter 0)
+		(color 0 0 0 0)
+	)
+	(no_connect
+		(at 250.19 107.95)
+	)
+	(no_connect
+		(at 248.92 123.19)
+	)
+	(no_connect
+		(at 213.36 118.11)
+	)
 	(wire
 		(pts
@@
 	(wire
 		(pts
+			(xy 204.47 55.88) (xy 212.09 55.88)
+		)
+		(stroke
+			(width 0)
+			(type default)
+		)
+	)
+	(wire
+		(pts
 			(xy 66.04 138.43) (xy 66.04 144.78)
 		)
@@
 	(wire
 		(pts
+			(xy 212.09 55.88) (xy 212.09 63.5)
+		)
+		(stroke
+			(width 0)
+			(type default)
+		)
+	)
+	(wire
+		(pts
 			(xy 52.07 182.88) (xy 69.85 182.88)
 		)
@@
 	(wire
 		(pts
+			(xy 196.85 55.88) (xy 191.77 55.88)
+		)
+		(stroke
+			(width 0)
+			(type default)
+		)
+	)
+	(wire
+		(pts
 			(xy 128.27 165.1) (xy 130.81 165.1)
 		)
@@
 	(wire
 		(pts
+			(xy 191.77 55.88) (xy 191.77 63.5)
+		)
+		(stroke
+			(width 0)
+			(type default)
+		)
+	)
+	(wire
+		(pts
 			(xy 165.1 95.25) (xy 171.45 95.25)
 		)
@@
 			)
 		)
-		(property "Value" "10u"
+		(property "Value" "47u"
 			(at 270.002 111.506 0)
 			(show_name no)
@@
 			)
 		)
-		(property "Footprint" "Capacitor_SMD:C_0805_2012Metric"
+		(property "Footprint" "Capacitor_THT:C_Radial_D5.0mm_H11.0mm_P2.00mm"
 			(at 268.9352 109.22 0)
 			(hide yes)
@@
 			)
 		)
-		(property "Value" "1u"
+		(property "Value" "100n"
 			(at 206.756 61.976 90)
 			(show_name no)
@@
 					(unit 1)
 				)
+			)
+		)
+	)
+	(symbol
+		(lib_id "Device:C")
+		(at 200.66 55.88 90)
+		(unit 1)
+		(body_style 1)
+		(exclude_from_sim no)
+		(in_bom yes)
+		(on_board yes)
+		(in_pos_files yes)
+		(dnp no)
+		(property "Reference" "C27"
+			(at 206.756 51.816 90)
+			(show_name no)
+			(do_not_autoplace no)
+			(effects
+				(font
+					(size 1.27 1.27)
+				)
+			)
+		)
+		(property "Value" "100n"
+			(at 206.756 54.356 90)
+			(show_name no)
+			(do_not_autoplace no)
+			(effects
+				(font
+					(size 1.27 1.27)
+				)
+			)
+		)
+		(property "Footprint" "Capacitor_SMD:C_0603_1608Metric"
+			(at 204.47 54.9148 0)
+			(hide yes)
+			(show_name no)
+			(do_not_autoplace no)
+			(effects
+				(font
+					(size 1.27 1.27)
+				)
+			)
+		)
+		(property "Datasheet" ""
+			(at 200.66 55.88 0)
+			(hide yes)
+			(show_name no)
+			(do_not_autoplace no)
+			(effects
+				(font
+					(size 1.27 1.27)
+				)
+			)
+		)
+		(property "Description" "Unpolarized capacitor"
+			(at 200.66 55.88 0)
+			(hide yes)
+			(show_name no)
+			(do_not_autoplace no)
+			(effects
+				(font
+					(size 1.27 1.27)
+				)
+			)
+		)
+		(pin "1"
+		)
+		(pin "2"
+		)
+		(instances
+			(project "DSP-hw"
+				(path "/5eaf86e8-787c-412f-bf3f-89f6d5971c5e"
+					(reference "C27")
+					(unit 1)
+				)

Commit message: sostituito dei componenti non piu disponibili
Parts:
- Q1: footprint Package_TO_SOT_THT:TO-92_Inline -> Package_TO_SOT_SMD:SOT-223-3_TabPin2
Changed lines of the file:
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@@
 			)
 		)
-		(property "Footprint" "Package_TO_SOT_THT:TO-92_Inline"
+		(property "Footprint" "Package_TO_SOT_SMD:SOT-223-3_TabPin2"
 			(at 231.14 40.005 0)
 			(hide yes)
@@
 			)
 		)
-		(property "Sim.Pins" "1=C 2=B 3=E"
+		(property "Sim.Pins" "1=B 2=C 3=E"
 			(at 236.22 41.91 0)
 			(hide yes)

Commit message: modifiche suggerite da osti
Parts:
- removed Y1: 12.228M, Crystal:Crystal_SMD_HC49-SD, symbol Device:Crystal
- added Y1: 12.228M, Crystal:Crystal_SMD_3225-4Pin_3.2x2.5mm, symbol Device:Crystal_GND24
- C22, C23: value 22p -> 18p
- R6: value 100 -> 80
Connections:
- net GND: now also Y1.2 (G), Y1.4 (G)
- net at C23.2, R6.1: now also Y1.3
- net at C22.2, U1.32 (MCLKI): now also Y1.1
Changed lines of the file:
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@@
 	(wire
 		(pts
+			(xy 179.07 100.33) (xy 176.53 100.33)
+		)
+		(stroke
+			(width 0)
+			(type default)
+		)
+	)
+	(wire
+		(pts
 			(xy 124.46 129.54) (xy 124.46 132.08)
 		)
@@
 	(wire
 		(pts
+			(xy 179.07 109.22) (xy 179.07 100.33)
+		)
+		(stroke
+			(width 0)
+			(type default)
+		)
+	)
+	(wire
+		(pts
 			(xy 109.22 135.89) (xy 111.76 135.89)
 		)
@@
 	)
 	(symbol
+		(lib_id "Device:Crystal_GND24")
+		(at 171.45 100.33 90)
+		(unit 1)
+		(body_style 1)
+		(exclude_from_sim no)
+		(in_bom yes)
+		(on_board yes)
+		(in_pos_files yes)
+		(dnp no)
+		(fields_autoplaced yes)
+		(property "Reference" "Y1"
+			(at 166.37 99.0599 90)
+			(show_name no)
+			(do_not_autoplace no)
+			(effects
+				(font
+					(size 1.27 1.27)
+				)
+				(justify left)
+			)
+		)
+		(property "Value" "12.228M"
+			(at 166.37 101.5999 90)
+			(show_name no)
+			(do_not_autoplace no)
+			(effects
+				(font
+					(size 1.27 1.27)
+				)
+				(justify left)
+			)
+		)
+		(property "Footprint" "Crystal:Crystal_SMD_3225-4Pin_3.2x2.5mm"
+			(at 171.45 100.33 0)
+			(hide yes)
+			(show_name no)
+			(do_not_autoplace no)
+			(effects
+				(font
+					(size 1.27 1.27)
+				)
+			)
+		)
+		(property "Datasheet" ""
+			(at 171.45 100.33 0)
+			(hide yes)
+			(show_name no)
+			(do_not_autoplace no)
+			(effects
+				(font
+					(size 1.27 1.27)
+				)
+			)
+		)
+		(property "Description" "Four pin crystal, GND on pins 2 and 4"
+			(at 171.45 100.33 0)
+			(hide yes)
+			(show_name no)
+			(do_not_autoplace no)
+			(effects
+				(font
+					(size 1.27 1.27)
+				)
+			)
+		)
+		(property private "KLC_S3.3" "The rectangle is not a symbol body but a graphical element"
+			(at 184.15 100.33 0)
+			(hide yes)
+			(show_name yes)
+			(do_not_autoplace no)
+			(effects
+				(font
+					(size 1.27 1.27)
+				)
+			)
+		)
+		(property private "KLC_S4.1" "Some pins are on 50mil grid to make the symbol small"
+			(at 186.69 100.33 0)
+			(hide yes)
+			(show_name yes)
+			(do_not_autoplace no)
+			(effects
+				(font
+					(size 1.27 1.27)
+				)
+			)
+		)
+		(pin "4"
+		)
+		(pin "1"
+		)
+		(pin "3"
+		)
+		(pin "2"
+		)
+		(instances
+			(project "DSP-hw"
+				(path "/5eaf86e8-787c-412f-bf3f-89f6d5971c5e"
+					(reference "Y1")
+					(unit 1)
+				)
+			)
+		)
+	)
+	(symbol
 		(lib_id "Memory_EEPROM:CAT24C256")
 		(at 140.97 176.53 0)
@@
 			)
 		)
-		(property "Value" "100"
+		(property "Value" "80"
 			(at 190.5 100.076 90)
 			(show_name no)
@@
 			)
 		)
-		(property "Value" "22p"
+		(property "Value" "18p"
 			(at 164.846 92.964 90)
 			(show_name no)
@@
 	)
 	(symbol
-		(lib_id "Device:Crystal")
-		(at 171.45 100.33 90)
-		(unit 1)
-		(body_style 1)
-		(exclude_from_sim no)
-		(in_bom yes)
-		(on_board yes)
-		(in_pos_files yes)
-		(dnp no)
-		(fields_autoplaced yes)
-		(property "Reference" "Y1"
-			(at 175.26 99.0599 90)
-			(show_name no)
-			(do_not_autoplace no)
-			(effects
-				(font
-					(size 1.27 1.27)
-				)
-				(justify right)
-			)
-		)
-		(property "Value" "12.228M"
-			(at 175.26 101.5999 90)
-			(show_name no)
-			(do_not_autoplace no)
-			(effects
-				(font
-					(size 1.27 1.27)
-				)
-				(justify right)
-			)
-		)
-		(property "Footprint" "Crystal:Crystal_SMD_HC49-SD"
-			(at 171.45 100.33 0)
-			(hide yes)
-			(show_name no)
-			(do_not_autoplace no)
-			(effects
-				(font
-					(size 1.27 1.27)
-				)
-			)
-		)
-		(property "Datasheet" ""
-			(at 171.45 100.33 0)
-			(hide yes)
-			(show_name no)
-			(do_not_autoplace no)
-			(effects
-				(font
-					(size 1.27 1.27)
-				)
-			)
-		)
-		(property "Description" "Two pin crystal"
-			(at 171.45 100.33 0)
-			(hide yes)
-			(show_name no)
-			(do_not_autoplace no)
-			(effects
-				(font
-					(size 1.27 1.27)
-				)
-			)
-		)
-		(pin "2"
-		)
-		(pin "1"
-		)
-		(instances
-			(project "DSP-hw"
-				(path "/5eaf86e8-787c-412f-bf3f-89f6d5971c5e"
-					(reference "Y1")
-					(unit 1)
-				)
-			)
-		)
-	)
-	(symbol
 		(lib_id "Transistor_FET:AO3400A")
 		(at 46.99 97.79 0)
@@
 			)
 		)
-		(property "Value" "22p"
+		(property "Value" "18p"
 			(at 165.1 110.744 90)
 			(show_name no)
@@
 					(unit 1)
 				)
+			)
+		)
+	)
+	(symbol
+		(lib_id "power:GND")
+		(at 179.07 109.22 0)
+		(unit 1)
+		(body_style 1)
+		(exclude_from_sim no)
+		(in_bom yes)
+		(on_board yes)
+		(in_pos_files yes)
+		(dnp no)
+		(fields_autoplaced yes)
+		(property "Reference" "#PWR067"
+			(at 179.07 115.57 0)
+			(hide yes)
+			(show_name no)
+			(do_not_autoplace no)
+			(effects
+				(font
+					(size 1.27 1.27)
+				)
+			)
+		)
+		(property "Value" "GND"
+			(at 179.07 114.3 0)
+			(show_name no)
+			(do_not_autoplace no)
+			(effects
+				(font
+					(size 1.27 1.27)
+				)
+			)
+		)
+		(property "Footprint" ""
+			(at 179.07 109.22 0)
+			(hide yes)
+			(show_name no)
+			(do_not_autoplace no)
+			(effects
+				(font
+					(size 1.27 1.27)
+				)
+			)
+		)
+		(property "Datasheet" ""
+			(at 179.07 109.22 0)
+			(hide yes)
+			(show_name no)
+			(do_not_autoplace no)
+			(effects
+				(font
+					(size 1.27 1.27)
+				)
+			)
+		)
+		(property "Description" "Power symbol creates a global label with name \"GND\" , ground"
+			(at 179.07 109.22 0)
+			(hide yes)
+			(show_name no)
+			(do_not_autoplace no)
+			(effects
+				(font
+					(size 1.27 1.27)
+				)
+			)
+		)
+		(pin "1"
+		)
+		(instances
+			(project "DSP-hw"
+				(path "/5eaf86e8-787c-412f-bf3f-89f6d5971c5e"
+					(reference "#PWR067")
+					(unit 1)
+				)

Commit message: messa apposto la silkscreen
Parts:
- added C5: 100n, Capacitor_SMD:C_0603_1608Metric, symbol Device:C
Connections:
- net GND: now also C5.2
- net at C3.1, C4.1, Q1.1 (C)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: now also C5.1
Changed lines of the file:
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@@
 	)
 	(junction
+		(at 254 63.5)
+		(diameter 0)
+		(color 0 0 0 0)
+	)
+	(junction
 		(at 254 41.91)
 		(diameter 0)
@@
 	)
 	(junction
+		(at 233.68 55.88)
+		(diameter 0)
+		(color 0 0 0 0)
+	)
+	(junction
 		(at 251.46 138.43)
 		(diameter 0)
@@
 	(wire
 		(pts
-			(xy 233.68 46.99) (xy 233.68 63.5)
+			(xy 233.68 46.99) (xy 233.68 55.88)
 		)
 		(stroke
@@
 	(wire
 		(pts
+			(xy 246.38 55.88) (xy 254 55.88)
+		)
+		(stroke
+			(width 0)
+			(type default)
+		)
+	)
+	(wire
+		(pts
 			(xy 156.21 172.72) (xy 158.75 172.72)
 		)
@@
 	(wire
 		(pts
+			(xy 233.68 55.88) (xy 233.68 63.5)
+		)
+		(stroke
+			(width 0)
+			(type default)
+		)
+	)
+	(wire
+		(pts
 			(xy 156.21 177.8) (xy 158.75 177.8)
 		)
@@
 	(wire
 		(pts
+			(xy 233.68 55.88) (xy 238.76 55.88)
+		)
+		(stroke
+			(width 0)
+			(type default)
+		)
+	)
+	(wire
+		(pts
 			(xy 60.96 102.87) (xy 60.96 107.95)
 		)
@@
 	(wire
 		(pts
+			(xy 254 55.88) (xy 254 63.5)
+		)
+		(stroke
+			(width 0)
+			(type default)
+		)
+	)
+	(wire
+		(pts
 			(xy 264.16 115.57) (xy 264.16 114.3)
 		)
@@
 					(unit 1)
 				)
+			)
+		)
+	)
+	(symbol
+		(lib_id "Device:C")
+		(at 242.57 55.88 90)
+		(unit 1)
+		(body_style 1)
+		(exclude_from_sim no)
+		(in_bom yes)
+		(on_board yes)
+		(in_pos_files yes)
+		(dnp no)
+		(property "Reference" "C5"
+			(at 248.666 51.816 90)
+			(show_name no)
+			(do_not_autoplace no)
+			(effects
+				(font
+					(size 1.27 1.27)
+				)
+			)
+		)
+		(property "Value" "100n"
+			(at 248.666 54.356 90)
+			(show_name no)
+			(do_not_autoplace no)
+			(effects
+				(font
+					(size 1.27 1.27)
+				)
+			)
+		)
+		(property "Footprint" "Capacitor_SMD:C_0603_1608Metric"
+			(at 246.38 54.9148 0)
+			(hide yes)
+			(show_name no)
+			(do_not_autoplace no)
+			(effects
+				(font
+					(size 1.27 1.27)
+				)
+			)
+		)
+		(property "Datasheet" ""
+			(at 242.57 55.88 0)
+			(hide yes)
+			(show_name no)
+			(do_not_autoplace no)
+			(effects
+				(font
+					(size 1.27 1.27)
+				)
+			)
+		)
+		(property "Description" "Unpolarized capacitor"
+			(at 242.57 55.88 0)
+			(hide yes)
+			(show_name no)
+			(do_not_autoplace no)
+			(effects
+				(font
+					(size 1.27 1.27)
+				)
+			)
+		)
+		(pin "1"
+		)
+		(pin "2"
+		)
+		(instances
+			(project "DSP-hw"
+				(path "/5eaf86e8-787c-412f-bf3f-89f6d5971c5e"
+					(reference "C5")
+					(unit 1)
+				)

Commit message: bom completata
Parts:
- removed Q1: BC327, Package_TO_SOT_SMD:SOT-223-3_TabPin2, symbol Transistor_BJT:BC327
- added Q1: BCX52, Package_TO_SOT_SMD:SOT-89-3, symbol Transistor_BJT:BCX52
Connections:
- net +3V3: now also Q1.2 (C)
- net at C3.1, C4.1, C5.1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: now also Q1.3 (E)
- net at R1.1, U1.17 (VDRIVE): now also Q1.1 (B)

Commit message: pulito lo schematico e fatto dei check
Parts:
- added R36: 2k2, Resistor_SMD:R_0603_1608Metric, symbol Device:R
- Q1: value BCX52 -> 2SA1013
- U2: value CAT24C256 -> CAT24C512
Connections:
- net +3V3: now also C27.2, C7.2, C8.2, Q1.3 (E), U1.34 (PVDD), U1.36 (AVDD), U1.48 (AVDD), R36.2; no longer Q1.2 (C)
- net CM: now reaches C16.1, C17.1, U1.40 (CM)
- net +1V8: now reaches C3.1, C4.1, C5.1, U1.13 (DVDD), U1.24 (DVDD)
- net +1V8: now also Q1.2 (C); no longer Q1.3 (E)
- net V_Drive: now reaches Q1.1 (B), R1.1, U1.17 (VDRIVE)
- net FiltA: now reaches C14.1, C15.1, U1.47 (FILTA)
- net FiltD: now reaches C12.1, C13.1, U1.41 (FILTD)
- net at U1.20 (ADDR1/CDATA/WB): now also R36.1
- no-connect marks 3 -> 2
Other:
- note added: "3V3 Supply"
- note added: "ADAU1701"
- note added: "DSP Led"
- note added: "EEPROM"
- note added: "PLL Filter"
- note added: "Potetiometer"
- note added: "Write Protection"
- moved on the sheet: C10, C11, C18, C19, C20, C21, C22, C23, C46, C47, C9, D3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
