File: DSP-hw.kicad_pcb (KiCad board)
At the start: 4 copper layers, 174.2 x 65.6 mm, 101 parts, among them J1 NC3MAH, J10 AudioJack3, J11 AudioJack3, J2 NC3MAH, J3 NC3MAH, J4 NC3MAH, J5 XLR3_AudioJack3_Combo_Ground, J6 XLR3_AudioJack3_Combo_Ground, J7 USB_C_Receptacle_USB2.0_16P, J8 Conn_01x04_Pin, J9 Conn_01x06_Pin, Q1 BC327, Q2 AO3400A, SW1 SW_Push, SW6 SW_SPST, SW7 SW_SPST, SW8 SW_Push, U1 ADAU1701, U2 CAT24C256, U3 AMS1117-3.3, U4 STM32F411RETx, Y1 12.228M

Commit message: recuperata versione di ieri
Parts:
- removed C1, C6: 100n, Capacitor_SMD:C_0603_1608Metric
- removed C2, C5: 10u, Capacitor_SMD:C_0603_1608Metric
- removed the R27 at (150.6, 62.1)
- removed the R31 at (150.6, 69.6)
- added C30: 4.7u, Capacitor_THT:C_Radial_D4.0mm_H7.0mm_P1.50mm, F.Cu at (132.5, 89.0)
- added C33: 100n, Capacitor_SMD:C_0603_1608Metric, F.Cu at (114.0, 81.5)
- added C36: 100n, Capacitor_SMD:C_0603_1608Metric, F.Cu at (117.0, 63.5)
- added C45: 100n, Capacitor_SMD:C_0603_1608Metric, F.Cu at (127.2, 65.0)
- added C48: 4.7u, Capacitor_SMD:C_0603_1608Metric, F.Cu at (139.5, 74.5)
- added JP1: SolderJumper_2_Open, Jumper:SolderJumper-2_P1.3mm_Open_TrianglePad1.0x1.5mm, F.Cu at (112.5, 73.2)
- added JP2: SolderJumper_2_Open, Jumper:SolderJumper-2_P1.3mm_Open_TrianglePad1.0x1.5mm, F.Cu at (115.0, 73.2)
- added JP3: SolderJumper_2_Open, Jumper:SolderJumper-2_P1.3mm_Open_TrianglePad1.0x1.5mm, F.Cu at (117.5, 73.2)
- added JP4: SolderJumper_2_Open, Jumper:SolderJumper-2_P1.3mm_Open_TrianglePad1.0x1.5mm, F.Cu at (120.0, 73.2)
- added SW2: SW_Push, Button_Switch_SMD:SW_SPST_PTS645Sx43SMTR92, F.Cu at (103.0, 73.0)
- added U5: TME-0505S, Converter_DCDC:Converter_DCDC_TRACO_TME_03xxS_05xxS_12xxS_Single_THT, F.Cu at (127.2, 85.8)
- added U6: ADUM3160, Package_SO:SOIC-16W_7.5x10.3mm_P1.27mm, F.Cu at (116.5, 73.3)
- C10, C11, C13, C15, C17, C4, C8: footprint Capacitor_SMD:C_0603_1608Metric -> Capacitor_SMD:C_0805_2012Metric
- C19, C20: footprint Capacitor_SMD:C_0603_1608Metric -> Capacitor_THT:C_Radial_D5.0mm_H11.0mm_P2.00mm
- C24, C25, C26, C29, C32: footprint Capacitor_SMD:C_0603_1608Metric -> Capacitor_SMD:C_1210_3225Metric
- C40: footprint Capacitor_SMD:C_0603_1608Metric -> Capacitor_THT:C_Radial_D4.0mm_H7.0mm_P1.50mm
- moved C25 133.9 mm to (218.5, 62.0), turned to -90 degrees
- moved R12 126.0 mm to (218.5, 66.3), turned to 90 degrees
- moved R11 122.9 mm to (215.5, 57.0)
- moved R9 111.0 mm to (199.5, 63.5)
- moved C24 104.4 mm to (189.0, 56.5), turned to -90 degrees
- moved R10 101.8 mm to (190.0, 61.0)
- moved C35 75.9 mm to (163.7, 52.0)
- moved R22 72.5 mm to (168.3, 52.0)
- moved C37 71.7 mm to (159.0, 52.0)
- moved R24 69.8 mm to (165.5, 54.5)
- moved C19 68.1 mm to (138.0, 88.5), turned to -90 degrees
- moved C21 65.2 mm to (141.0, 84.5)
- moved C18 65.1 mm to (141.0, 78.5)
- moved C20 62.0 mm to (144.0, 88.5), turned to -90 degrees
- moved SW8 61.7 mm to (159.0, 90.5), turned to 180 degrees
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Connections:
- J7 pad A1: GND -> GNDA
- J7 pad A12: GND -> GNDA
- J7 pad A4: +5V -> +5VA
- J7 pad A9: +5V -> +5VA
- J7 pad B1: GND -> GNDA
- J7 pad B12: GND -> GNDA
- J7 pad B4: +5V -> +5VA
- J7 pad B9: +5V -> +5VA
- J7 pad SH: GND -> GNDA
- Q1 pad 2: +3V3 -> Net-(Q1-B)
- R1 pad 1: +3V3 -> Net-(Q1-B)
- R25 pad 2: GND -> GNDA
- R26 pad 2: GND -> GNDA
- U1 pad 17: +3V3 -> Net-(Q1-B)
- U4 pad 30: unconnected-(U4-VCAP1-Pad30) -> Net-(U4-VCAP1)
- U4 pad 60: unconnected-(U4-BOOT0-Pad60) -> GND
- U4 pad 7: unconnected-(U4-NRST-Pad7) -> Net-(U4-NRST)
Routing:
- added copper zone on B.Cu, net GND
- added copper zone on F.Cu, net GND
- added copper zone on In1.Cu, net GND
- added copper zone on In2.Cu, net GND
Other:
- board size 174.2 x 65.6 mm -> 184 x 65.6 mm

Commit message: routing iniziale
Parts:
- C35: footprint Capacitor_SMD:C_0603_1608Metric -> Capacitor_SMD:C_1210_3225Metric
- moved Q1 44.4 mm to (198.8, 86.7), turned to 180 degrees
- moved SW2 43.0 mm to (143.7, 59.2), turned to 0 degrees
- moved R21 32.6 mm to (133.0, 51.7), turned to -90 degrees
- moved C34 28.2 mm to (130.3, 50.9), turned to 180 degrees
- moved C9 25.6 mm to (202.6, 87.1)
- moved R8 25.0 mm to (183.0, 84.7), turned to 90 degrees
- moved C11 24.2 mm to (207.7, 69.4)
- moved C12 24.2 mm to (198.2, 69.2)
- moved C13 24.2 mm to (200.2, 69.4)
- moved C14 24.2 mm to (194.2, 69.2)
- moved C15 24.2 mm to (196.2, 69.4)
- moved C16 24.2 mm to (205.2, 69.4)
- moved C17 24.2 mm to (202.7, 69.4)
- moved C3 24.2 mm to (205.2, 87.1)
- moved C4 24.2 mm to (207.2, 87.1)
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Routing:
- net /SCL: track 0.00 -> 114.2 mm
- net /SDA: track 0.00 -> 63.0 mm
- net +5VA: track 0.00 -> 47.3 mm
- net Net-(C24-Pad1): track 0.00 -> 27.3 mm
- net Net-(C25-Pad1): track 0.00 -> 27.0 mm
- net /Micro/D+: track 0.00 -> 18.8 mm, vias 0 -> 1
- net /Micro/D-: track 0.00 -> 18.4 mm
- net Net-(J6-Pad1): track 0.00 -> 18.1 mm
- net Net-(J5-Pad1): track 0.00 -> 18.1 mm
- net Net-(Q1-C): track 0.00 -> 11.6 mm
- net Net-(U6-PDEN): track 0.00 -> 11.5 mm
- net Net-(J7-CC1): track 0.00 -> 11.0 mm, vias 0 -> 1
- net Net-(Q1-B): track 0.00 -> 9.97 mm
- net Net-(C37-Pad1): track 0.00 -> 8.38 mm
- net Net-(C31-Pad1): track 0.00 -> 8.15 mm
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- added copper zone on In1.Cu, net +3V3
- added copper zone on In2.Cu, net +3V3
- added copper zone on B.Cu, net GNDA
- added copper zone on F.Cu, net GNDA
- removed copper zone on In2.Cu, net GND
