File: DSP-hw.kicad_pcb (KiCad board)
At the start: 2 copper layers, 185 x 66.6 mm, 120 parts, among them J1 NC3MAH, J10 AudioJack3, J11 AudioJack3, J2 NC3MAH, J3 NC3MAH, J4 NC3MAH, J5 XLR3_AudioJack3_Combo_Ground, J6 XLR3_AudioJack3_Combo_Ground, J7 USB_C_Receptacle_USB2.0_16P, J8 Conn_01x04_Pin, J9 Conn_01x06_Pin, Q1 BCX52, Q2 AO3400A, SW1 SW_Push, SW2 SW_Push, SW6 SW_SPST, SW7 SW_SPST, SW8 SW_Push, U1 ADAU1701, U2 CAT24C256, U3 AMS1117-3.3, U4 STM32F411RETx, U5 TME-0505S, U6 ADUM3160, Y1 12.228M, Y2 8M

Commit message: pulito lo schematico e fatto dei check
Parts:
- added H5: MountingHole, MountingHole:MountingHole_2.2mm_M2_Pad_Via, F.Cu at (222.0, 64.0)
- added H6: MountingHole, MountingHole:MountingHole_2.2mm_M2_Pad_Via, F.Cu at (222.0, 80.0)
- added H7: MountingHole, MountingHole:MountingHole_2.2mm_M2_Pad_Via, F.Cu at (240.0, 59.5)
- added H8: MountingHole, MountingHole:MountingHole_2.2mm_M2_Pad_Via, F.Cu at (240.0, 84.0)
- added J12: Conn_01x06_Socket, Connector_PinHeader_2.54mm:PinHeader_1x06_P2.54mm_Vertical, F.Cu at (241.0, 78.0)
- added R20: 33, Resistor_SMD:R_0603_1608Metric, F.Cu at (116.4, 85.3)
- added R23: 33, Resistor_SMD:R_0603_1608Metric, F.Cu at (117.9, 85.3)
- added R36: 2k2, Resistor_SMD:R_0603_1608Metric, F.Cu at (201.6, 88.0)
- added R37: 33, Resistor_SMD:R_0603_1608Metric, F.Cu at (119.9, 65.3)
- added R38: 33, Resistor_SMD:R_0603_1608Metric, F.Cu at (118.3, 65.3)
- Q1: value BCX52 -> 2SA1013
- U2: value CAT24C256 -> CAT24C512
- moved R25 6.30 mm to (124.3, 93.7)
- moved SW2 1.90 mm to (124.7, 58.5)
- moved J8 1.80 mm to (220.0, 90.0)
- moved R26 1.26 mm to (124.3, 92.2)
- moved G*** 0.57 mm to (90.0, 66.5)
- moved C9 0.40 mm to (202.2, 85.0)
- moved C3 0.28 mm to (205.1, 84.8)
- moved R1 0.28 mm to (200.6, 85.0)
Connections:
- net Net-(C24-Pad1) renamed /Input Output/1 Hot
- net Net-(C25-Pad1) renamed /Input Output/0 Hot
- net Net-(Q1-B) renamed /V_Drive
- net Net-(SW6-B) renamed /Input Output/1 Cold
- net Net-(SW7-B) renamed /Input Output/0 Cold
- net Net-(U1-CM) renamed /CM
- net Net-(U1-FILTA) renamed /FiltA
- net Net-(U1-FILTD) renamed /FiltD
- C27 pad 2: Net-(U1-PVDD) -> +3V3
- C3 pad 1: Net-(Q1-E) -> +1V8
- C4 pad 1: Net-(Q1-E) -> +1V8
- C5 pad 1: Net-(Q1-E) -> +1V8
- C7 pad 2: Net-(U1-PVDD) -> +3V3
- C8 pad 2: Net-(U1-PVDD) -> +3V3
- J7 pad A6: /Micro/D+ -> Net-(J7-D+-PadA6)
- J7 pad A7: /Micro/D- -> Net-(J7-D--PadA7)
- J7 pad B6: /Micro/D+ -> Net-(J7-D+-PadA6)
- J7 pad B7: /Micro/D- -> Net-(J7-D--PadA7)
- Q1 pad 2: +3V3 -> +1V8
- Q1 pad 3: Net-(Q1-E) -> +3V3
- U1 pad 13: Net-(Q1-E) -> +1V8
- U1 pad 20: unconnected-(U1-ADDR1/CDATA/WB-Pad20) -> Net-(U1-ADDR1/CDATA/WB)
- U1 pad 24: Net-(Q1-E) -> +1V8
- U1 pad 34: Net-(U1-PVDD) -> +3V3
- U1 pad 36: Net-(U1-PVDD) -> +3V3
- U1 pad 48: Net-(U1-PVDD) -> +3V3
- U6 pad 10: /Micro/D+ iso -> Net-(U6-DD+)
- U6 pad 11: /Micro/D- iso -> Net-(U6-DD-)
Routing:
- net +5V: track 39.3 -> 161.3 mm, vias 1 -> 2
- net /Input Output/1 Cold: track 9.01 -> 63.1 mm
- net /Input Output/1 Hot: track 27.5 -> 78.0 mm
- net +3V3: track 464.8 -> 490.8 mm
- net /Input Output/0 Hot: track 27.0 -> 52.3 mm
- net Net-(U1-PVDD): track 24.3 -> 0.00 mm
- net Net-(Q1-E): track 24.2 -> 0.00 mm, vias 2 -> 0
- net +1V8: track 0.00 -> 23.5 mm, vias 0 -> 2
- net /Input Output/0 Cold: track 9.44 -> 32.7 mm
- net /Micro/D+: track 20.8 -> 11.7 mm
- net /Micro/D-: track 20.6 -> 11.8 mm
- net Net-(J7-D--PadA7): track 0.00 -> 7.25 mm
- net Net-(J7-D+-PadA6): track 0.00 -> 7.06 mm
- net Net-(U1-ADDR1/CDATA/WB): track 0.00 -> 6.49 mm
- net Net-(U6-DD-): track 0.00 -> 3.13 mm
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Other:
- board text added: "D+"
- board text added: "D-"
- board text added: "Phanthom +48V board"
- board text added: "V1.0 Rev 07/08/2026"
- board text removed: "V1.0 Rev 03/08/2026"
