File: micro.kicad_sch (KiCad schematic)
At the start: 17 parts, among them J7 USB_C_Receptacle_USB2.0_16P, J8 Conn_01x04_Pin, J9 Conn_01x06_Pin, U4 STM32G473CETx

Commit message: errore alla coca
Parts:
- removed U4: STM32G473CETx, Package_QFP:LQFP-48_7x7mm_P0.5mm, symbol MCU_ST_STM32G4:STM32G473CETx
- added C45: 100n, Capacitor_SMD:C_0603_1608Metric, symbol Device:C
- added C48: 4.7u, Capacitor_SMD:C_0603_1608Metric, symbol Device:C
- added SW2: SW_Push, symbol Switch:SW_Push
- added U4: STM32F411RETx, Package_QFP:LQFP-64_10x10mm_P0.5mm, symbol MCU_ST_STM32F4:STM32F411RETx
Connections:
- net +3V3: now also U4.1 (VBAT), U4.13 (VDDA), U4.19 (VDD), U4.32 (VDD), U4.48 (VDD), U4.64 (VDD)
- net BCLK_1: now also U4.20 (PA4)
- net BCLK_2: now also U4.33 (PB12)
- net D+: now also U4.45 (PA12)
- net D-: now also U4.44 (PA11)
- net DIN: now also U4.23 (PA7)
- net DOUT: now also U4.11 (PC3)
- net GND: now also C45.2, C48.2, SW2.2, U4.12 (VSSA), U4.18 (VSS), U4.31 (VSS), U4.47 (VSS), U4.60 (BOOT0), U4.63 (VSS)
- net LRCK_1: now also U4.21 (PA5)
- net LRCK_2: now also U4.29 (PB10)
- net SCL: now also U4.58 (PB6)
- net SDA: now also U4.59 (PB7)
- net SWCLK: now also U4.49 (PA14)
- net SWDIO: now also U4.46 (PA13)
- net UART1_RX: now also U4.42 (PA9)
- net UART1_TX: now also U4.43 (PA10)
- net WP: now also U4.57 (PB5)
- net at R27.1: now also U4.3 (PC14)
- net at R31.1: now also U4.4 (PC15)
- new net: C45.1, SW2.1, U4.7 (NRST)
- new net: C48.1, U4.30 (VCAP1)

Commit message: recuperata versione di ieri
Parts:
- added C30: 4.7u, Capacitor_THT:C_Radial_D4.0mm_H7.0mm_P1.50mm, symbol Device:C
- added C33, C36: 100n, Capacitor_SMD:C_0603_1608Metric, symbol Device:C
- added JP1, JP2, JP3, JP4: SolderJumper_2_Open, Jumper:SolderJumper-2_P1.3mm_Open_TrianglePad1.0x1.5mm, symbol Jumper:SolderJumper_2_Open
- added U5: TME-0505S, Converter_DCDC:Converter_DCDC_TRACO_TME_03xxS_05xxS_12xxS_Single_THT, symbol Converter_DCDC:TME-0505S
- added U6: ADUM3160, Package_SO:SOIC-16W_7.5x10.3mm_P1.27mm, symbol Interface_USB:ADUM3160
- C40: footprint Capacitor_SMD:C_0603_1608Metric -> Capacitor_THT:C_Radial_D4.0mm_H7.0mm_P1.50mm
- SW2: footprint (none) -> Button_Switch_SMD:SW_SPST_PTS645Sx43SMTR92
Connections:
- net +5V: now also JP1.2 (B), U5.4 (+Vout), U6.16 (VBUS2); no longer J7.A4 (VBUS), J7.A9 (VBUS), J7.B4 (VBUS), J7.B9 (VBUS)
- net D+: now also JP3.1 (A), U6.7 (UD+)
- net D-: now also JP2.1 (A), U6.6 (UD-)
- net GND: now also C36.2, JP4.2 (B), U5.3 (-Vout), U6.15 (GND2), U6.9 (GND2); no longer J7.A1 (GND), J7.A12 (GND), J7.B1 (GND), J7.B12 (GND), J7.SH (SHIELD), R25.2, R26.2
- new net: C36.1, U6.12 (PIN), U6.13 (SPD), U6.14 (VDD2)
- new net: C33.1, U6.3 (VDD1), U6.4 (PDEN), U6.5 (SPU)
- new net +5VA: C30.1, J7.A4 (VBUS), J7.A9 (VBUS), J7.B4 (VBUS), J7.B9 (VBUS), JP1.1 (A), U5.2 (+Vin), U6.1 (VBUS1)
- new net D+ iso: JP3.2 (B), U6.10 (DD+)
- new net D- iso: JP2.2 (B), U6.11 (DD-)
- new net GNDA: C30.2, C33.2, J7.A1 (GND), J7.A12 (GND), J7.B1 (GND), J7.B12 (GND), J7.SH (SHIELD), JP4.1 (A), R25.2, R26.2, U5.1 (-Vin), U6.2 (GND1), U6.8 (GND1)
Other:
- moved on the sheet: C45, C48, D1, D2, J7, R25, R26, R27, R31, SW2, U4

Commit message: routing iniziale
Other:
- moved on the sheet: C33, C45, SW2
Changed lines of the file:
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@@
 	)
 	(junction
-		(at 82.55 85.09)
-		(diameter 0)
-		(color 0 0 0 0)
-	)
-	(junction
 		(at 38.1 76.2)
 		(diameter 0)
@@
 	)
 	(junction
-		(at 80.01 175.26)
+		(at 82.55 95.25)
 		(diameter 0)
 		(color 0 0 0 0)
 	)
 	(junction
-		(at 76.2 95.25)
+		(at 80.01 175.26)
 		(diameter 0)
 		(color 0 0 0 0)
@@
 	)
 	(junction
-		(at 196.85 69.85)
+		(at 247.65 157.48)
 		(diameter 0)
 		(color 0 0 0 0)
 	)
 	(junction
-		(at 247.65 157.48)
+		(at 194.31 69.85)
 		(diameter 0)
 		(color 0 0 0 0)
@@
 	)
 	(junction
-		(at 196.85 72.39)
+		(at 82.55 85.09)
 		(diameter 0)
 		(color 0 0 0 0)
@@
 	(wire
 		(pts
-			(xy 181.61 69.85) (xy 196.85 69.85)
-		)
-		(stroke
-			(width 0)
-			(type default)
-		)
-	)
-	(wire
-		(pts
-			(xy 76.2 97.79) (xy 76.2 95.25)
+			(xy 82.55 97.79) (xy 82.55 95.25)
 		)
 		(stroke
@@
 	(wire
 		(pts
-			(xy 196.85 69.85) (xy 228.6 69.85)
+			(xy 182.88 69.85) (xy 194.31 69.85)
 		)
 		(stroke
@@
 	(wire
 		(pts
+			(xy 194.31 69.85) (xy 194.31 72.39)
+		)
+		(stroke
+			(width 0)
+			(type default)
+		)
+	)
+	(wire
+		(pts
 			(xy 60.96 44.45) (xy 63.5 44.45)
 		)
@@
 	(wire
 		(pts
-			(xy 196.85 83.82) (xy 189.23 83.82)
+			(xy 194.31 83.82) (xy 189.23 83.82)
 		)
 		(stroke
@@
 	(wire
 		(pts
-			(xy 82.55 95.25) (xy 76.2 95.25)
-		)
-		(stroke
-			(width 0)
-			(type default)
-		)
-	)
-	(wire
-		(pts
 			(xy 69.85 148.59) (xy 69.85 151.13)
 		)
@@
 	(wire
 		(pts
-			(xy 82.55 85.09) (xy 82.55 86.36)
-		)
-		(stroke
-			(width 0)
-			(type default)
-		)
-	)
-	(wire
-		(pts
 			(xy 71.12 177.8) (xy 71.12 173.99)
 		)
@@
 	(wire
 		(pts
-			(xy 181.61 82.55) (xy 181.61 83.82)
+			(xy 182.88 81.28) (xy 182.88 83.82)
 		)
 		(stroke
@@
 	(wire
 		(pts
-			(xy 196.85 72.39) (xy 196.85 69.85)
-		)
-		(stroke
-			(width 0)
-			(type default)
-		)
-	)
-	(wire
-		(pts
 			(xy 82.55 69.85) (xy 82.55 85.09)
 		)
@@
 	(wire
 		(pts
-			(xy 196.85 72.39) (xy 196.85 73.66)
-		)
-		(stroke
-			(width 0)
-			(type default)
-		)
-	)
-	(wire
-		(pts
 			(xy 82.55 69.85) (xy 88.9 69.85)
 		)
@@
 	(wire
 		(pts
-			(xy 196.85 83.82) (xy 196.85 82.55)
+			(xy 194.31 83.82) (xy 194.31 82.55)
 		)
 		(stroke
@@
 	(wire
 		(pts
+			(xy 194.31 69.85) (xy 228.6 69.85)
+		)
+		(stroke
+			(width 0)
+			(type default)
+		)
+	)
+	(wire
+		(pts
 			(xy 72.39 44.45) (xy 82.55 44.45)
 		)
@@
 	(wire
 		(pts
-			(xy 181.61 74.93) (xy 181.61 69.85)
+			(xy 182.88 73.66) (xy 182.88 69.85)
 		)
 		(stroke
@@
 	(wire
 		(pts
-			(xy 38.1 95.25) (xy 76.2 95.25)
+			(xy 38.1 95.25) (xy 82.55 95.25)
 		)
 		(stroke
@@
 	(wire
 		(pts
-			(xy 82.55 93.98) (xy 82.55 95.25)
+			(xy 82.55 92.71) (xy 82.55 95.25)
 		)
 		(stroke
@@
 	(wire
 		(pts
-			(xy 189.23 83.82) (xy 181.61 83.82)
+			(xy 189.23 83.82) (xy 182.88 83.82)
 		)
 		(stroke
@@
 	(symbol
 		(lib_id "Device:C")
-		(at 181.61 78.74 0)
+		(at 182.88 77.47 0)
 		(unit 1)
 		(body_style 1)
@@
 		(dnp no)
 		(property "Reference" "C45"
-			(at 184.658 72.39 0)
+			(at 176.276 76.2 0)
 			(show_name no)
 			(do_not_autoplace no)
@@
 		)
 		(property "Value" "100n"
-			(at 184.658 74.93 0)
+			(at 176.276 78.74 0)
 			(show_name no)
 			(do_not_autoplace no)
@@
 		)
 		(property "Footprint" "Capacitor_SMD:C_0603_1608Metric"
-			(at 182.5752 82.55 0)
+			(at 183.8452 81.28 0)
 			(hide yes)
 			(show_name no)
@@
 		)
 		(property "Datasheet" ""
-			(at 181.61 78.74 0)
+			(at 182.88 77.47 0)
 			(hide yes)
 			(show_name no)
@@
 		)
 		(property "Description" "Unpolarized capacitor"
-			(at 181.61 78.74 0)
+			(at 182.88 77.47 0)
 			(hide yes)
 			(show_name no)
@@
 	(symbol
 		(lib_id "Device:C")
-		(at 82.55 90.17 0)
+		(at 82.55 88.9 0)
 		(unit 1)
 		(body_style 1)
@@
 		(dnp no)
 		(property "Reference" "C33"
-			(at 74.168 89.154 0)
+			(at 74.168 87.884 0)
 			(show_name no)
 			(do_not_autoplace no)
@@
 		)
 		(property "Value" "100n"
-			(at 74.168 91.694 0)
+			(at 74.168 90.424 0)
 			(show_name no)
 			(do_not_autoplace no)
@@
 		)
 		(property "Footprint" "Capacitor_SMD:C_0603_1608Metric"
-			(at 83.5152 93.98 0)
+			(at 83.5152 92.71 0)
 			(hide yes)
 			(show_name no)
@@
 		)
 		(property "Datasheet" ""
-			(at 82.55 90.17 0)
+			(at 82.55 88.9 0)
 			(hide yes)
 			(show_name no)
@@
 		)
 		(property "Description" "Unpolarized capacitor"
-			(at 82.55 90.17 0)
+			(at 82.55 88.9 0)
 			(hide yes)
 			(show_name no)
@@
 	(symbol
 		(lib_id "Switch:SW_Push")
-		(at 196.85 77.47 270)
+		(at 194.31 77.47 270)
 		(unit 1)
 		(body_style 1)
@@
 		(fields_autoplaced yes)
 		(property "Reference" "SW2"
-			(at 200.66 76.1999 90)
+			(at 198.12 76.1999 90)
 			(show_name no)
 			(do_not_autoplace no)
@@
 		)
 		(property "Value" "SW_Push"
-			(at 200.66 78.7399 90)
+			(at 198.12 78.7399 90)
 			(show_name no)
 			(do_not_autoplace no)
@@
 		)
 		(property "Footprint" "Button_Switch_SMD:SW_SPST_PTS645Sx43SMTR92"
-			(at 201.93 77.47 0)
+			(at 199.39 77.47 0)
 			(hide yes)
 			(show_name no)
@@
 		)
 		(property "Datasheet" ""
-			(at 201.93 77.47 0)
+			(at 199.39 77.47 0)
 			(hide yes)
 			(show_name no)
@@
 		)
 		(property "Description" "Push button switch, generic, two pins"
-			(at 196.85 77.47 0)
+			(at 194.31 77.47 0)
 			(hide yes)
 			(show_name no)
@@
 	(symbol
 		(lib_id "power:GNDA")
-		(at 76.2 97.79 0)
+		(at 82.55 97.79 0)
 		(unit 1)
 		(body_style 1)
@@
 		(fields_autoplaced yes)
 		(property "Reference" "#PWR035"
-			(at 76.2 104.14 0)
+			(at 82.55 104.14 0)
 			(hide yes)
 			(show_name no)
@@
 		)
 		(property "Value" "GNDA"
-			(at 76.2 102.87 0)
+			(at 82.55 102.87 0)
 			(show_name no)
 			(do_not_autoplace no)
@@
 		)
 		(property "Footprint" ""
-			(at 76.2 97.79 0)
+			(at 82.55 97.79 0)
 			(hide yes)
 			(show_name no)
@@
 		)
 		(property "Datasheet" ""
-			(at 76.2 97.79 0)
+			(at 82.55 97.79 0)
 			(hide yes)
 			(show_name no)
@@
 		)
 		(property "Description" "Power symbol creates a global label with name \"GNDA\" , analog ground"
-			(at 76.2 97.79 0)
+			(at 82.55 97.79 0)
 			(hide yes)
 			(show_name no)
