File: _restore_backup_2026-07-27T17-27-44-474/DSP-hw.kicad_pcb (KiCad board)
At the start: 4 copper layers, 184 x 65.6 mm, 107 parts, among them J1 NC3MAH, J10 AudioJack3, J11 AudioJack3, J2 NC3MAH, J3 NC3MAH, J4 NC3MAH, J5 XLR3_AudioJack3_Combo_Ground, J6 XLR3_AudioJack3_Combo_Ground, J7 USB_C_Receptacle_USB2.0_16P, J8 Conn_01x04_Pin, J9 Conn_01x06_Pin, Q1 BC327, Q2 AO3400A, SW1 SW_Push, SW2 SW_Push, SW6 SW_SPST, SW7 SW_SPST, SW8 SW_Push, U1 ADAU1701, U2 CAT24C256, U3 AMS1117-3.3, U4 STM32F411RETx, U5 TME-0505S, U6 ADUM3160, Y1 12.228M

Commit message: routing praticamente fatto forse
Parts:
- J7: footprint Connector_USB:USB_C_Receptacle_GCT_USB4105-xx-A_16P_TopMnt_Horizontal -> Connector_USB:USB_C_Receptacle_GCT_USB4085
- moved JP1 19.2 mm to (112.5, 73.2), turned to 90 degrees
- moved JP4 18.8 mm to (120.3, 73.2), turned to 90 degrees
- moved J7 5.38 mm to (113.0, 88.3)
- moved C30 0.36 mm to (127.5, 83.0)
- moved R27 0.20 mm to (105.5, 87.0)
- moved J11 0.11 mm to (62.5, 74.0)
- moved J10 0.10 mm to (62.5, 61.0)
Routing:
- net +5VA: track 41.0 -> 48.8 mm, vias 2 -> 0
- net GNDA: track 3.19 -> 10.4 mm, vias 4 -> 2
- net GND: track 64.8 -> 60.6 mm
- net +5V: track 42.0 -> 38.7 mm
- net /Micro/D-: track 19.3 -> 18.4 mm
- net /MP9: track 150.6 -> 151.3 mm
- net /Micro/D- iso: track 56.1 -> 55.5 mm
- net /Micro/D+: track 18.9 -> 18.8 mm, vias 0 -> 1
- net Net-(J7-CC1): track 11.1 -> 11.0 mm, vias 2 -> 1
- net Net-(J7-CC2): track 7.20 -> 7.21 mm, vias 0 -> 1
