File: _restore_backup_2026-07-27T17-27-44-474/DSP-hw.kicad_sch (KiCad schematic)
At the start: 46 parts, among them Q1 BC327, Q2 AO3400A, SW1 SW_Push, SW8 SW_Push, U1 ADAU1701, U2 CAT24C256, U3 AMS1117-3.3, Y1 12.228M

Commit message: routing praticamente fatto forse
Connections:
- net MP1: now reaches U1.10 (MP1)
- net MP1: now also R34.1
- net MP3: no longer names the net of U1.28 (MP3)
- net MP3: no longer R34.1
Changed lines of the file:
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@@
-	(wire
-		(pts
-			(xy 248.92 113.03) (xy 250.19 113.03)
-		)
-		(stroke
-			(width 0)
-			(type default)
-		)
-	)
 	(wire
 		(pts
@@
 		)
 	)
+	(label "MP1"
+		(at 250.19 107.95 0)
+		(effects
+			(font
+				(size 1.27 1.27)
+			)
+			(justify left bottom)
+		)
+	)
 	(label "DAC3"
 		(at 52.07 33.02 0)
@@
 		)
 	)
-	(label "BCLK_2"
+	(label "BCLK__2"
 		(at 73.66 30.48 180)
 		(effects
@@
 		)
 	)
-	(label "MP3"
-		(at 250.19 113.03 0)
-		(effects
-			(font
-				(size 1.27 1.27)
-			)
-			(justify left bottom)
-		)
-	)
 	(label "BCLK_2"
 		(at 250.19 133.35 0)
@@
 		)
 	)
-	(label "MP3"
+	(label "MP1"
 		(at 91.44 133.35 0)
 		(effects
