File: _restore_backup_2026-07-27T17-27-44-474/micro.kicad_sch (KiCad schematic)
At the start: 29 parts, among them J7 USB_C_Receptacle_USB2.0_16P, J8 Conn_01x04_Pin, J9 Conn_01x06_Pin, SW2 SW_Push, U4 STM32F411RETx, U5 TME-0505S, U6 ADUM3160

Commit message: routing praticamente fatto forse
Parts:
- J7: footprint Connector_USB:USB_C_Receptacle_GCT_USB4105-xx-A_16P_TopMnt_Horizontal -> Connector_USB:USB_C_Receptacle_GCT_USB4085
Connections:
- net D+: now also U4.45 (PA12)
- net D+ iso: no longer U4.45 (PA12)
- net D-: now also U4.44 (PA11)
- net D- iso: no longer U4.44 (PA11)
- net SWCLK: now also J9.3 (Pin_3); no longer J9.2 (Pin_2)
- net SWDIO: now also J9.2 (Pin_2); no longer J9.3 (Pin_3)
- net WP: now also U4.57 (PB5); no longer U4.17 (PA3)
Changed lines of the file:
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@@
 	(wire
 		(pts
-			(xy 264.16 77.47) (xy 267.97 77.47)
-		)
-		(stroke
-			(width 0)
-			(type default)
-		)
-	)
-	(wire
-		(pts
 			(xy 30.48 173.99) (xy 36.83 173.99)
 		)
@@
 	(wire
 		(pts
+			(xy 264.16 125.73) (xy 266.7 125.73)
+		)
+		(stroke
+			(width 0)
+			(type default)
+		)
+	)
+	(wire
+		(pts
 			(xy 60.96 44.45) (xy 60.96 45.72)
 		)
@@
 		)
 	)
-	(label "D+ iso"
+	(label "D+"
 		(at 267.97 100.33 0)
 		(effects
@@
 		)
 	)
-	(label "SWCLK"
-		(at 30.48 179.07 180)
-		(effects
-			(font
-				(size 1.27 1.27)
-			)
-			(justify right bottom)
-		)
-	)
 	(label "D- iso"
 		(at 71.12 128.27 0)
@@
 		)
 	)
-	(label "D-"
-		(at 85.09 80.01 0)
+	(label "SWCLK"
+		(at 30.48 176.53 180)
 		(effects
 			(font
 				(size 1.27 1.27)
 			)
-			(justify left bottom)
+			(justify right bottom)
 		)
 	)
-	(label "SWDIO"
-		(at 30.48 176.53 180)
+	(label "D-"
+		(at 85.09 80.01 0)
 		(effects
 			(font
 				(size 1.27 1.27)
 			)
-			(justify right bottom)
+			(justify left bottom)
 		)
 	)
@@
 		)
 	)
+	(label "SWDIO"
+		(at 30.48 179.07 180)
+		(effects
+			(font
+				(size 1.27 1.27)
+			)
+			(justify right bottom)
+		)
+	)
 	(label "UART1_RX"
 		(at 267.97 92.71 0)
@@
 		)
 	)
-	(label "D- iso"
+	(label "D-"
 		(at 267.97 97.79 0)
 		(effects
@@
 		)
 	)
+	(hierarchical_label "WP"
+		(shape input)
+		(at 266.7 125.73 0)
+		(effects
+			(font
+				(size 1.27 1.27)
+			)
+			(justify left)
+		)
+	)
 	(hierarchical_label "SCL"
 		(shape input)
@@
 		)
 	)
-	(hierarchical_label "WP"
-		(shape input)
-		(at 267.97 77.47 0)
-		(effects
-			(font
-				(size 1.27 1.27)
-			)
-			(justify left)
-		)
-	)
 	(hierarchical_label "DOUT"
 		(shape input)
@@
 			)
 		)
-		(property "Footprint" "Connector_USB:USB_C_Receptacle_GCT_USB4105-xx-A_16P_TopMnt_Horizontal"
+		(property "Footprint" "Connector_USB:USB_C_Receptacle_GCT_USB4085"
 			(at 41.91 53.34 0)
 			(hide yes)
